File: hardware/125b/125b.kicad_pcb (KiCad board)
At the start: 2 copper layers, 59 x 75 mm, 49 parts, among them J1 Guitar in, J2 Barrel_Jack, J3 Conn_02x05_Odd_Even_MountingP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, J4 Guitar out, SW1 SW_Push_SPDT, SW2 RotaryEncoder_Switch, SW3 SW_Push, SW4 SW_Push, U1 L78L05_TO92, U2 TL074

Commit message: Name change from Crouds to Prog1 on PCB
Other:
- board text added: "Prog1 v0.6 Denis Crowdy, Prog Pedals"
- board text removed: "Crouds v0.6 Denis Crowdy, Prog Pedals"
Changed lines of the file:
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@@
 			)
 		)
-		(model "/home/dcrowdy/progpedals/crouds/hardware/3dmodels/3-D NMJ6HCD2.stp"
+		(model "/Users/dcrowdy/progpedals/crouds/hardware/3dmodels/3-D NMJ6HCD2.stp"
 			(offset
 				(xyz -4 -8 0.5)
@@
 		(layer "Edge.Cuts")
 	)
-	(gr_text "Crouds v0.6 Denis Crowdy, Prog Pedals"
-		(at 146.5 108.45 0)
+	(gr_text "Prog1 v0.6 Denis Crowdy, Prog Pedals"
+		(at 142 108.45 0)
 		(layer "B.SilkS")
 		(effects
