File: hardware/footswitch/footswitch.kicad_sch (KiCad schematic)
At the start: 6 parts, among them J1 Conn_02x05_Counter_Clockwise

Commit message: Adjust footprint for dpdt alpha
Parts:
- S1, S2: footprint pcb switch:SF12011F010220RM050 -> pcb switch:DPDT momentary footswitch
Changed lines of the file:
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@@
 			)
 		)
-		(property "Footprint" "pcb switch:SF12011F010220RM050"
+		(property "Footprint" "pcb switch:DPDT momentary footswitch"
 			(at 139.7 157.15 0)
 			(effects
@@
 			)
 		)
-		(property "Footprint" "pcb switch:SF12011F010220RM050"
+		(property "Footprint" "pcb switch:DPDT momentary footswitch"
 			(at 139.7 143.18 0)
 			(effects

Commit message: Adjust footprints for Tayda compact footswitches
Parts:
- 3DPDT Footswitch1: footprint Button_Switch_THT:Switches_Stomp_Switch_3PDT -> Library:0.7 footswitches - 3dpdt tayda
- S1, S2: footprint pcb switch:DPDT momentary footswitch -> Library:0.7 footswitches
Changed lines of the file:
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@@
 			)
 		)
-		(property "Footprint" "pcb switch:DPDT momentary footswitch"
+		(property "Footprint" "Library:0.7 footswitches"
 			(at 139.7 157.15 0)
 			(effects
@@
 			)
 		)
-		(property "Footprint" "Button_Switch_THT:Switches_Stomp_Switch_3PDT"
+		(property "Footprint" "Library:0.7 footswitches - 3dpdt tayda"
 			(at 133.35 100.33 0)
 			(effects
@@
 			)
 		)
-		(property "Footprint" "pcb switch:DPDT momentary footswitch"
+		(property "Footprint" "Library:0.7 footswitches"
 			(at 139.7 143.18 0)
 			(effects
